File: Eagle/PLACA Mina.brd (EAGLE design)
At the start: 106.3 x 77.5 mm, 25 parts

Commit message: adi;'oes
Parts:
- removed TENSAO: (no value), Robotica-IFRN-SC-conectores:6410-02
- moved R3 7.62 mm to (96.5, 3.81)
- moved SERVO.1 5.24 mm to (55.9, 22.9), turned to 0 degrees
- moved LED3 2.54 mm to (96.5, 8.89)
- moved S4 1.27 mm to (27.9, 6.35)
- moved SERVO.2 1.27 mm to (66.0, 22.9), turned to 0 degrees
- moved PONTE-H 1.27 mm to (34.3, 68.6)
Connections:
- net +5V: no longer TENSAO.1
- net GND: no longer TENSAO.2
Routing:
- net +5V: track 170.9 -> 204.0 mm
- net GND: track 29.7 -> 20.3 mm
- net N$17: track 9.00 -> 0.00 mm
- net N$16: track 9.00 -> 0.00 mm
- net N$15: track 9.00 -> 0.00 mm
- net N$22: track 18.1 -> 11.7 mm
- net N$21: track 15.5 -> 9.94 mm
- net N$26: track 18.6 -> 23.5 mm
- net N$31: track 8.67 -> 5.68 mm
- net N$28: track 15.8 -> 13.5 mm
- net N$29: track 11.2 -> 9.19 mm
- net N$23: track 12.9 -> 14.8 mm
- net N$25: track 14.1 -> 12.2 mm
- net N$9: track 7.62 -> 6.35 mm
- net N$8: track 7.62 -> 6.35 mm
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Other:
- board size 106.3 x 77.5 mm -> 106.3 x 76.2 mm
